File: pcb-v1.kicad_sch (KiCad schematic)
At the start: 32 parts, among them J1 Conn_01x03_Socket, J10 Screw_Terminal_01x04, J11 Screw_Terminal_01x04, J12 Screw_Terminal_01x04, J13 Screw_Terminal_01x04, J14 Screw_Terminal_01x06, J15 Conn_01x06_Pin, J2 Conn_01x03_Socket, J3 Conn_01x03_Socket, J4 Conn_01x03_Socket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

Commit message: wiring complete
Connections:
- net 5VDC: now also A1.5V2 (SPI_5V)
- no-connect marks 70 -> 69
Changed lines of the file:
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@@
-	)
-	(no_connect
-		(at 160.02 27.94)
 	)
 	(no_connect
@@
 		(pts
 			(xy 95.25 41.91) (xy 95.25 54.61)
+		)
+		(stroke
+			(width 0)
+			(type default)
+		)
+	)
+	(wire
+		(pts
+			(xy 160.02 24.13) (xy 160.02 27.94)
 		)
 		(stroke
@@
 		)
 	)
+	(label "5VDC"
+		(at 160.02 24.13 180)
+		(effects
+			(font
+				(size 1.27 1.27)
+			)
+			(justify right bottom)
+		)
+	)
